File: kicad/nrf24l01_breakout.kicad_pcb (KiCad board)
At the start: 2 copper layers, 26.7 x 31.8 mm, 6 parts, among them P1 CONN_02X04, P2 CONN_01X08, P3 CONN_01X08

Commit message: Revision 2.0 - Smaller
Parts:
- moved REF** 11.5 mm to (168.9, 97.8)
- moved C1 10.2 mm to (163.8, 114.3)
- moved C2 8.13 mm to (161.3, 109.2)
- moved P1 7.18 mm to (163.8, 104.1)
Routing:
- net Net-(C1-Pad2): track 37.2 -> 27.6 mm
- net Net-(P1-Pad8): track 23.7 -> 17.6 mm
- net Net-(P1-Pad7): track 20.1 -> 15.0 mm
- net Net-(P1-Pad6): track 22.6 -> 18.6 mm
- net Net-(P1-Pad5): track 19.1 -> 16.1 mm
- net Net-(P1-Pad4): track 22.6 -> 19.7 mm
- net Net-(P1-Pad3): track 20.1 -> 17.1 mm
Other:
- board size 26.7 x 31.8 mm -> 22.9 x 24.1 mm
- board text added: "Antenna this way"
- board text added: "nRF24L01+ breakout board Rev 2.0 by Arnaud Boudou"
- board text removed: "nRF24L01+ breakout board Rev 1.0 © Arnaud Boudou"
